File: Project_Acoustic_Detector/Project_Acoustic_Detector.kicad_pcb (KiCad board)
At the start: 2 copper layers, 50.5 x 46 mm, 41 parts, among them J1 Conn_01x04_Pin, J3 Conn_02x03_Top_Bottom, J4 Conn_02x03_Top_Bottom, J5 Conn_02x03_Top_Bottom, J6 USB_C_Receptacle_USB2.0_16P, J7 Micro_SD_Card_Det2, SW1 SW_Push, SW2 SW_Push, U1 ESP32-S3-WROOM-1, U2 AMS1117-3.3

Commit message: updated KiCad project
Parts:
- removed C14: 10u, Capacitor_Tantalum_SMD:CP_EIA-3216-18_Kemet-A_HandSolder
- removed R13, R14, R15: 10k, Resistor_SMD:R_1206_3216Metric_Pad1.30x1.75mm_HandSolder
- removed R16, R4: 100k, Resistor_SMD:R_1206_3216Metric_Pad1.30x1.75mm_HandSolder
- added J10: Conn_01x03_Pin, Connector_PinHeader_2.54mm:PinHeader_1x03_P2.54mm_Vertical, F.Cu at (116.0, 87.6)
- added J11: Conn_01x03_Pin, Connector_PinHeader_2.54mm:PinHeader_1x03_P2.54mm_Vertical, F.Cu at (116.1, 100.1)
- added J12: Conn_01x03_Pin, Connector_PinHeader_2.54mm:PinHeader_1x03_P2.54mm_Vertical, F.Cu at (116.0, 113.0)
- added J2: Conn_01x03_Pin, Connector_PinHeader_2.54mm:PinHeader_1x03_P2.54mm_Vertical, F.Cu at (112.0, 87.5)
- added J666: Conn_01x04_Pin, Connector_PinHeader_2.54mm:PinHeader_1x04_P2.54mm_Vertical, F.Cu at (1.79, 1.79)
- added J8: Conn_01x05_Pin, Connector_PinHeader_2.54mm:PinHeader_1x05_P2.54mm_Vertical, F.Cu at (125.0, 99.5)
- added J9: Conn_01x05_Pin, Connector_PinHeader_2.54mm:PinHeader_1x05_P2.54mm_Vertical, F.Cu at (147.0, 109.7)
- J3, J4: value Conn_02x03_Top_Bottom -> Conn_01x03_Pin; footprint Connector_PinHeader_2.54mm:PinHeader_2x03_P2.54mm_Vertical -> Connector_PinHeader_2.54mm:PinHeader_1x03_P2.54mm_Vertical
- J5: value Conn_02x03_Top_Bottom -> Conn_01x05_Pin; footprint Connector_PinHeader_2.54mm:PinHeader_2x03_P2.54mm_Vertical -> Connector_PinHeader_2.54mm:PinHeader_1x05_P2.54mm_Vertical
- moved J5 45.8 mm to (168.0, 115.1), turned to 180 degrees
- moved C5 30.9 mm to (108.5, 86.5), turned to -90 degrees
- moved C6 26.6 mm to (108.5, 112.0), turned to -90 degrees
- moved C7 24.3 mm to (108.5, 99.0), turned to -90 degrees
- moved J4 22.0 mm to (112.0, 113.1), turned to 180 degrees
- moved J3 17.4 mm to (112.0, 100.1), turned to 180 degrees
- moved C10 13.5 mm to (131.5, 98.9)
- moved C11 13.5 mm to (131.5, 101.4)
- moved C12 13.5 mm to (124.0, 105.9)
- moved C13 13.5 mm to (126.5, 105.9)
- moved C8 13.5 mm to (139.0, 109.0)
- moved C9 13.5 mm to (136.5, 108.9)
- moved D1 13.5 mm to (121.5, 117.4)
- moved FB1 13.5 mm to (125.0, 110.4)
- moved J6 13.5 mm to (131.5, 118.4)
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Connections:
- C12 pad 1: /+3.3V_Audio -> +3.3V_Audio
- C13 pad 2: /+3.3V_Audio -> +3.3V_Audio
- C5 pad 1: /+3.3V_Audio -> +3.3V_Audio
- C6 pad 1: /+3.3V_Audio -> +3.3V_Audio
- C7 pad 1: /+3.3V_Audio -> +3.3V_Audio
- C8 pad 1: +5V -> GND
- C8 pad 2: GND -> +5V
- FB1 pad 2: /+3.3V_Audio -> +3.3V_Audio
- J3 pad 2: /+3.3V_Audio -> +3.3V_Audio
- J3 pad 3: /I2S_SD2 -> /I2S_SD1
- J4 pad 2: /+3.3V_Audio -> +3.3V_Audio
- J4 pad 3: /I2S_SD1 -> /I2S_SD2
- J5 pad 2: /+3.3V_Audio -> +3.3V_Audio
- J5 pad 3: /I2S_SD1 -> /I2S_SD2
- J5 pad 4: GND -> /I2S_WS
- J5 pad 5: /I2S_WS -> /I2S_SCK
Routing:
- net +3.3V: track 0.00 -> 145.5 mm, vias 0 -> 7
- net /I2S_SCK: track 0.00 -> 96.6 mm, vias 0 -> 4
- net /I2S_WS: track 0.00 -> 95.1 mm, vias 0 -> 4
- net +3.3V_Audio: track 0.00 -> 92.6 mm, vias 0 -> 1
- net GND: track 0.00 -> 68.7 mm, vias 0 -> 2
- net /I2S_SD1: track 0.00 -> 50.4 mm, vias 0 -> 3
- net /BOOT0: track 0.00 -> 39.4 mm
- net /SD_DET: track 0.00 -> 37.2 mm
- net +5V: track 0.00 -> 35.8 mm
- net /I2S_SD2: track 0.00 -> 28.6 mm
- net /USB_D-: track 0.00 -> 27.9 mm
- net /USB_D+: track 0.00 -> 26.1 mm
- net /SD_CS: track 0.00 -> 25.8 mm
- net /SD_CLK: track 0.00 -> 25.3 mm
- net /Indicator: track 0.00 -> 24.7 mm, vias 0 -> 2
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Other:
- board size 50.5 x 46 mm -> 63 x 46 mm

Commit message: updated KiCad project
Parts:
- removed C5, C6, C7: 100n, Capacitor_SMD:C_1206_3216Metric_Pad1.33x1.80mm_HandSolder
- removed J10, J11, J12, J2, J3, J4: Conn_01x03_Pin, Connector_PinHeader_2.54mm:PinHeader_1x03_P2.54mm_Vertical
- removed J666: Conn_01x04_Pin, Connector_PinHeader_2.54mm:PinHeader_1x04_P2.54mm_Vertical
- added C14: 10u, Capacitor_Tantalum_SMD:CP_EIA-3216-18_Kemet-A_HandSolder, F.Cu at (159.0, 105.5)
- C4: value 10n -> 100n
- J6: footprint Connector_USB:USB_C_Receptacle_HRO_TYPE-C-31-M-12 -> Connector_USB:USB_C_Receptacle_GCT_USB4085
- moved D1 23.3 mm to (137.8, 100.8), turned to 180 degrees
- moved R2 17.9 mm to (137.8, 103.4)
- moved R11 14.9 mm to (123.6, 117.7), turned to 180 degrees
- moved C4 7.20 mm to (160.3, 90.6)
- moved R9 7.20 mm to (156.8, 90.5)
- moved D2 6.30 mm to (166.3, 90.7)
- moved R3 6.30 mm to (163.8, 90.7)
- moved J6 5.79 mm to (128.5, 113.5)
- moved R8 5.27 mm to (139.4, 115.6), turned to 0 degrees
- moved R10 2.41 mm to (123.6, 115.2), turned to 180 degrees
- moved R7 2.35 mm to (139.4, 118.0), turned to 0 degrees
- moved C10 1.44 mm to (131.5, 97.5), turned to 180 degrees
- moved C11 1.44 mm to (131.5, 100.0), turned to 180 degrees
- moved C12 1.44 mm to (124.0, 104.5)
- moved C13 1.44 mm to (126.5, 104.5)
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Connections:
- C10 pad 1: GND -> +3.3V
- C10 pad 2: +3.3V -> GND
- C11 pad 1: GND -> +3.3V
- C11 pad 2: +3.3V -> GND
- C8 pad 1: GND -> +5V
- C8 pad 2: +5V -> GND
Routing:
- net /I2S_SCK: track 96.6 -> 65.2 mm, vias 4 -> 0
- net /I2S_WS: track 95.1 -> 66.2 mm, vias 4 -> 0
- net +3.3V: track 145.5 -> 125.5 mm, vias 7 -> 4
- net /EN: track 19.0 -> 34.2 mm, vias 3 -> 0
- net /Indicator: track 24.7 -> 37.3 mm
- net /BOOT0: track 39.4 -> 29.1 mm
- net Net-(J6-D+-PadA6): track 20.5 -> 12.1 mm, vias 2 -> 1
- net /USB_D-: track 27.9 -> 35.6 mm
- net /I2S_SD2: track 28.6 -> 35.6 mm, vias 0 -> 1
- net /I2S_SD1: track 50.4 -> 43.7 mm, vias 3 -> 0
- net Net-(J6-D--PadA7): track 18.7 -> 13.1 mm, vias 0 -> 1
- net +3.3V_Audio: track 92.6 -> 97.2 mm, vias 1 -> 0
- net /SD_CS: track 25.8 -> 22.1 mm
- net /SD_DET: track 37.2 -> 40.8 mm
- net /USB_D+: track 26.1 -> 29.2 mm
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- added copper zone on B.Cu, net GND
- added copper zone on F.Cu, net GND
Other:
- board size 63 x 46 mm -> 50.5 x 46 mm
