File: Project_Acoustic_Detector/Project_Acoustic_Detector.kicad_sch (KiCad schematic)
At the start: 41 parts, among them J1 Conn_01x04_Pin, J3 Conn_02x03_Top_Bottom, J4 Conn_02x03_Top_Bottom, J5 Conn_02x03_Top_Bottom, J6 USB_C_Receptacle_USB2.0_16P, J7 Micro_SD_Card_Det2, SW1 SW_Push, SW2 SW_Push, U1 ESP32-S3-WROOM-1, U2 AMS1117-3.3

Commit message: updated KiCad project
Parts:
- removed J3, J4, J5: Conn_02x03_Top_Bottom, Connector_PinHeader_2.54mm:PinHeader_2x03_P2.54mm_Vertical, symbol Connector_Generic:Conn_02x03_Top_Bottom
- removed R13, R14, R15: 10k, Resistor_SMD:R_1206_3216Metric_Pad1.30x1.75mm_HandSolder, symbol Device:R
- removed R16, R4: 100k, Resistor_SMD:R_1206_3216Metric_Pad1.30x1.75mm_HandSolder, symbol Device:R
- added J10, J11, J12, J2, J3, J4: Conn_01x03_Pin, Connector_PinHeader_2.54mm:PinHeader_1x03_P2.54mm_Vertical, symbol Connector:Conn_01x03_Pin
- added J5, J8, J9: Conn_01x05_Pin, Connector_PinHeader_2.54mm:PinHeader_1x05_P2.54mm_Vertical, symbol Connector:Conn_01x05_Pin
- added J666: Conn_01x04_Pin, Connector_PinHeader_2.54mm:PinHeader_1x04_P2.54mm_Vertical, symbol Connector:Conn_01x04_Pin
Connections:
- net +3.3V_Audio: now also J11.1 (Pin_1), J2.2 (Pin_2), J3.2 (Pin_2), J4.2 (Pin_2), J5.2 (Pin_2), J8.2 (Pin_2), J9.2 (Pin_2)
- net +5V: now also C8.2; no longer C8.1
- net GND: now also C8.1, J10.1 (Pin_1), J12.1 (Pin_1), J2.1 (Pin_1), J3.1 (Pin_1), J4.1 (Pin_1), J5.1 (Pin_1), J8.1 (Pin_1), J9.1 (Pin_1); no longer C8.2
- net I2S_SCK: now also J10.3 (Pin_3), J11.3 (Pin_3), J12.3 (Pin_3), J5.5 (Pin_5), J8.5 (Pin_5), J9.5 (Pin_5)
- net I2S_SD1: now also J2.3 (Pin_3), J3.3 (Pin_3), J8.3 (Pin_3), J9.3 (Pin_3)
- net I2S_SD2: now also J4.3 (Pin_3), J5.3 (Pin_3)
- net I2S_WS: now also J10.2 (Pin_2), J11.2 (Pin_2), J12.2 (Pin_2), J5.4 (Pin_4), J8.4 (Pin_4), J9.4 (Pin_4)
- no-connect marks 25 -> 29
Other:
- note added: "Conn_Mic1"
- note added: "Conn_Mic2"
- note added: "Conn_Mic3"
- moved on the sheet: C8, D1, D2, R12, R2, R3

Commit message: updated KiCad project
Parts:
- removed C5, C6, C7: 100n, Capacitor_SMD:C_1206_3216Metric_Pad1.33x1.80mm_HandSolder, symbol Device:C
- removed J10, J11, J12, J2, J3, J4: Conn_01x03_Pin, Connector_PinHeader_2.54mm:PinHeader_1x03_P2.54mm_Vertical, symbol Connector:Conn_01x03_Pin
- removed J666: Conn_01x04_Pin, Connector_PinHeader_2.54mm:PinHeader_1x04_P2.54mm_Vertical, symbol Connector:Conn_01x04_Pin
- C4: value 10n -> 100n
- J6: footprint Connector_USB:USB_C_Receptacle_HRO_TYPE-C-31-M-12 -> Connector_USB:USB_C_Receptacle_GCT_USB4085; PCS PartN (none) -> 00-00077751; Price (none) -> 50; Store (none) -> Cosmodrom
Connections:
- net +3.3V: now also C10.1, C11.1; no longer C10.2, C11.2
- net +5V: now also C8.1; no longer C8.2
- net GND: now also C10.2, C11.2, C8.2; no longer C10.1, C11.1, C8.1
- no-connect marks 29 -> 25
Other:
- note removed: "Mic1"
- note removed: "Mic2"
- note removed: "Mic3"
- moved on the sheet: C10, C11, C14, C8, C9, J1, J7
